File: qboards-template.kicad_pcb (KiCad board)
At the start: 2 copper layers, 10.2 x 15.2 mm, 4 parts

Commit message: Set default values for Page Settings, updated default and minimal board setup
Other:
- net class Default: clearance 0.1524 -> 0.2032; trace_width 0.1524 -> 0.2032
- net class Minimal added: clearance 0.1524, trace_width 0.1524, via_dia 0.8, via_drill 0.4
- rule trace_clearance: 0.1524 -> 0.2032
- board text removed: "Description of the board"
- board text removed: "QBoard Template [BRD_REF]"
Changed lines of the file:
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@@
   (general
     (thickness 1.2)
-    (drawings 26)
+    (drawings 24)
     (tracks 0)
     (zones 0)
@@
   )
   (page A4)
+  (title_block
+    (title BRD-REF)
+    (rev 1)
+    (company QBoards)
+    (comment 1 "Description of the board")
+  )
   (layers
     (0 F.Cu signal)
@@
   )
   (setup
-    (last_trace_width 0.1524)
-    (trace_clearance 0.1524)
+    (last_trace_width 0.2032)
+    (trace_clearance 0.2032)
     (zone_clearance 0.508)
     (zone_45_only no)
@@
     (solder_mask_min_width 0.25)
     (aux_axis_origin 0 0)
-    (visible_elements FFFFEF7F)
+    (visible_elements 7FFFFFFF)
     (pcbplotparams
       (layerselection 0x010fc_ffffffff)
@@
   (net 0 "")
   (net_class Default "This is the default net class."
+    (clearance 0.2032)
+    (trace_width 0.2032)
+    (via_dia 0.8)
+    (via_drill 0.4)
+    (uvia_dia 0.3)
+    (uvia_drill 0.1)
+  )
+  (net_class Minimal ""
     (clearance 0.1524)
     (trace_width 0.1524)
@@
   (gr_arc (start 148.336 109.982) (end 148.336 111.252) (angle -90) (layer Edge.Cuts) (width 0.05))
   (gr_arc (start 148.336 97.282) (end 149.606 97.282) (angle -90) (layer Edge.Cuts) (width 0.05))
-  (gr_text "QBoard Template [BRD_REF]" (at 109.728 189.484) (layer F.Fab)
-    (effects (font (size 1.5 1.5) (thickness 0.3)) (justify left mirror))
-  )
-  (gr_text "Description of the board" (at 117.602 168.91) (layer F.Fab)
-    (effects (font (size 1.5 1.5) (thickness 0.3)) (justify left mirror))
-  )
   (gr_line (start 148.336 111.252) (end 140.716 111.252) (layer Edge.Cuts) (width 0.05))
   (gr_line (start 149.606 97.282) (end 149.606 109.982) (layer Edge.Cuts) (width 0.05))
